File: ADAC-Shield.sch (EAGLE design)
At the start: 46 parts, among them U1 ARDUINO-MEGAFULL, U2 LM358D

Commit message: Schematic finished. Started designing a PCB. Added schematic image
Parts:
- added C21, C23, C25: 0.1, rcl:C-EUC0805
- added C22, C24, C26: 47, rcl:CPOL-EUA
- added C27, C28: 100, rcl:CPOL-EUB
- added JACK_OUT: ST-11M-0, smok:ST-11M-0
- added R17: 220, rcl:R-EU_R0805
- added R18, R19: 1, rcl:R-EU_R0805
- R8, R9: value 22k -> 1k
Connections:
- new net ADC_BCK: ADC.BCK
- new net ADC_DATAO: ADC.DATAO
- new net ADC_MSSEL: ADC.MSSEL
- new net ADC_PWON: ADC.PWON
- new net ADC_SFOR: ADC.SFOR
- new net ADC_SYSCLK: ADC.SYSCLK
- new net ADC_WS: ADC.WS
- new net N$19: ADC.VRP, C20.+, C21.2, R17.1
- new net N$20: ADC.VDDA, C23.1, C24.+, R18.1
- new net N$25: ADC.VDDD, C25.2, C26.+, R19.2
- net +3V3: now also C27.+, R19.1
- net GND: now also ADC.VRN, ADC.VSSA, ADC.VSSD, C20.-, C21.1, C22.-, C23.2, C24.-, C25.1, C26.-, C27.-, C28.-, JACK_OUT.SLEEVE; no longer C20.+
- net LEFT_DAC_OUT: now also JACK_OUT.TIP
- net N$18: now also C22.+; no longer C20.-
- net RIGHT_DAC_OUT: now also JACK_OUT.RING
- net V+: now also C28.+, R17.2, R18.2
Other:
- note removed: "NEED TO CHECK THIS PART"
- moved on the sheet: C20

Commit message: Some progress in PCB layout
Parts:
- removed R1: 0, rcl:R-EU_R1206
- added JP4: (no value), pinhead:PINHD-1X2
Connections:
- net +3V3: now also JP4.2; no longer R1.1
- net V+: now also JP4.1; no longer R1.2
Other:
- moved on the sheet: C21, C22
Changed lines of the file:
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@@
 <part name="+3V1" library="supply1" deviceset="+3V3" device=""/>
 <part name="P+2" library="supply1" deviceset="V+" device=""/>
-<part name="R1" library="rcl" deviceset="R-EU_" device="R1206" value="0"/>
 <part name="P+3" library="supply1" deviceset="V+" device=""/>
 <part name="C2" library="rcl" deviceset="C-EU" device="C0805" value="0.1"/>
@@
 <part name="JACK_OUT" library="smok" deviceset="ST-11M-0" device=""/>
 <part name="GND31" library="supply1" deviceset="GND" device=""/>
+<part name="JP4" library="pinhead" deviceset="PINHD-1X2" device=""/>
 </parts>
 <sheets>
@@
 <instance part="+3V1" gate="G$1" x="-180.34" y="73.66"/>
 <instance part="P+2" gate="1" x="-160.02" y="73.66"/>
-<instance part="R1" gate="G$1" x="-170.18" y="68.58"/>
 <instance part="P+3" gate="1" x="-60.96" y="93.98"/>
 <instance part="C2" gate="G$1" x="-60.96" y="83.82"/>
@@
 <instance part="GND17" gate="1" x="-104.14" y="-205.74"/>
 <instance part="C19" gate="G$1" x="-30.48" y="-157.48" rot="R180"/>
-<instance part="GND18" gate="1" x="-38.1" y="-162.56"/>
+<instance part="GND18" gate="1" x="-43.18" y="-162.56"/>
 <instance part="GND19" gate="1" x="-30.48" y="-162.56"/>
 <instance part="GND20" gate="1" x="-2.54" y="-162.56" rot="R270"/>
-<instance part="C21" gate="G$1" x="-30.48" y="-172.72" rot="R180"/>
+<instance part="C21" gate="G$1" x="-25.4" y="-172.72" rot="R180"/>
 <instance part="GND21" gate="1" x="-38.1" y="-177.8"/>
-<instance part="GND22" gate="1" x="-30.48" y="-177.8"/>
+<instance part="GND22" gate="1" x="-25.4" y="-177.8"/>
 <instance part="R17" gate="G$1" x="-45.72" y="-167.64" rot="R180"/>
 <instance part="P+7" gate="1" x="-53.34" y="-162.56"/>
@@
 <instance part="GND28" gate="1" x="40.64" y="-177.8" rot="R90"/>
 <instance part="C20" gate="G$1" x="-38.1" y="-170.18"/>
-<instance part="C22" gate="G$1" x="-38.1" y="-154.94"/>
+<instance part="C22" gate="G$1" x="-43.18" y="-154.94"/>
 <instance part="C27" gate="G$1" x="-180.34" y="66.04"/>
 <instance part="C28" gate="G$1" x="-160.02" y="66.04"/>
@@
 <instance part="JACK_OUT" gate="G$1" x="-93.98" y="-152.4"/>
 <instance part="GND31" gate="1" x="-106.68" y="-160.02"/>
+<instance part="JP4" gate="G$1" x="-170.18" y="60.96" rot="R270"/>
 </instances>
 <busses>
@@
 <pinref part="+3V1" gate="G$1" pin="+3V3"/>
 <wire x1="-180.34" y1="71.12" x2="-180.34" y2="68.58" width="0.1524" layer="91"/>
-<pinref part="R1" gate="G$1" pin="1"/>
-<wire x1="-180.34" y1="68.58" x2="-175.26" y2="68.58" width="0.1524" layer="91"/>
 <pinref part="C27" gate="G$1" pin="+"/>
 <junction x="-180.34" y="68.58"/>
+<pinref part="JP4" gate="G$1" pin="2"/>
+<wire x1="-180.34" y1="68.58" x2="-170.18" y2="68.58" width="0.1524" layer="91"/>
+<wire x1="-170.18" y1="68.58" x2="-170.18" y2="63.5" width="0.1524" layer="91"/>
 </segment>
 <segment>
@@
 <pinref part="P+2" gate="1" pin="V+"/>
 <wire x1="-160.02" y1="71.12" x2="-160.02" y2="68.58" width="0.1524" layer="91"/>
-<pinref part="R1" gate="G$1" pin="2"/>
-<wire x1="-160.02" y1="68.58" x2="-165.1" y2="68.58" width="0.1524" layer="91"/>
+<wire x1="-160.02" y1="68.58" x2="-167.64" y2="68.58" width="0.1524" layer="91"/>
 <pinref part="C28" gate="G$1" pin="+"/>
 <junction x="-160.02" y="68.58"/>
+<pinref part="JP4" gate="G$1" pin="1"/>
+<wire x1="-167.64" y1="68.58" x2="-167.64" y2="63.5" width="0.1524" layer="91"/>
 </segment>
 <segment>
@@
 <segment>
 <pinref part="C19" gate="G$1" pin="2"/>
-<wire x1="-38.1" y1="-152.4" x2="-30.48" y2="-152.4" width="0.1524" layer="91"/>
+<wire x1="-43.18" y1="-152.4" x2="-30.48" y2="-152.4" width="0.1524" layer="91"/>
 <pinref part="ADC" gate="G$1" pin="VREF"/>
 <wire x1="-30.48" y1="-152.4" x2="2.54" y2="-152.4" width="0.1524" layer="91"/>
@@
 <wire x1="-40.64" y1="-167.64" x2="-38.1" y2="-167.64" width="0.1524" layer="91"/>
 <pinref part="ADC" gate="G$1" pin="VRP"/>
-<wire x1="-38.1" y1="-167.64" x2="-30.48" y2="-167.64" width="0.1524" layer="91"/>
-<wire x1="-30.48" y1="-167.64" x2="2.54" y2="-167.64" width="0.1524" layer="91"/>
-<junction x="-30.48" y="-167.64"/>
+<wire x1="-38.1" y1="-167.64" x2="-25.4" y2="-167.64" width="0.1524" layer="91"/>
+<wire x1="-25.4" y1="-167.64" x2="2.54" y2="-167.64" width="0.1524" layer="91"/>
+<junction x="-25.4" y="-167.64"/>
 <pinref part="R17" gate="G$1" pin="1"/>
 <pinref part="C20" gate="G$1" pin="+"/>

Commit message: Board layout finished for v0.1
Parts:
- U1: device SparkFun-Boards:ARDUINO-MEGAFULL -> SparkFun-Boards_modified:ARDUINO-MEGAFULL
Connections:
- net ADC_BCK: now also U1.45
- net ADC_DATAO: now also U1.47
- net ADC_MSSEL: now also U1.48
- net ADC_PWON: now also U1.50
- net ADC_SFOR: now also U1.51
- net ADC_SYSCLK: now also U1.49
- net ADC_WS: now also U1.46
- net DAC_BCK: now also U1.34
- net DAC_DATAI: now also U1.36
- net DAC_DEEM: now also U1.40
- net DAC_MUTE: now also U1.39
- net DAC_PCS: now also U1.41
- net DAC_SFOR0: now also U1.38
- net DAC_SFOR1: now also U1.37
- net DAC_SYSCLK: now also U1.33
- net DAC_WS: now also U1.35
Other:
- note added: "PC1"
- note added: "PC12"
- note added: "PC13"
- note added: "PC14"
- note added: "PC15"
- note added: "PC16"
- note added: "PC17"
- note added: "PC18"
- note added: "PC2"
- note added: "PC3"
- note added: "PC4"
- note added: "PC5"
- note added: "PC6"
- note added: "PC7"
- note added: "PC8"
- note added: "PC9"
Changed lines of the file:
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@@
 </classes>
 <parts>
-<part name="U1" library="SparkFun-Boards" deviceset="ARDUINO-MEGA" device="FULL"/>
 <part name="U2" library="CircuitHub" deviceset="1680-LM358DT" device="" value="LM358D"/>
 <part name="GND1" library="supply1" deviceset="GND" device=""/>
@@
 <part name="GND31" library="supply1" deviceset="GND" device=""/>
 <part name="JP4" library="pinhead" deviceset="PINHD-1X2" device=""/>
+<part name="U1" library="SparkFun-Boards_modified" deviceset="ARDUINO-MEGA" device="FULL"/>
 </parts>
 <sheets>
@@
 <text x="-63.5" y="53.34" size="1.778" layer="91">Low Gain</text>
 <text x="-66.04" y="-2.54" size="1.778" layer="91">Low Gain</text>
+<text x="-198.12" y="0" size="1.778" layer="97">PC1</text>
+<text x="-198.12" y="-2.54" size="1.778" layer="97">PC2</text>
+<text x="-198.12" y="-5.08" size="1.778" layer="97">PC3</text>
+<text x="-198.12" y="-7.62" size="1.778" layer="97">PC4</text>
+<text x="-198.12" y="-10.16" size="1.778" layer="97">PC5</text>
+<text x="-198.12" y="-12.7" size="1.778" layer="97">PC6</text>
+<text x="-198.12" y="-15.24" size="1.778" layer="97">PC7</text>
+<text x="-198.12" y="-17.78" size="1.778" layer="97">PC8</text>
+<text x="-198.12" y="-20.32" size="1.778" layer="97">PC9</text>
+<text x="-198.12" y="-45.72" size="1.778" layer="97">PC12</text>
+<text x="-198.12" y="-43.18" size="1.778" layer="97">PC13</text>
+<text x="-198.12" y="-40.64" size="1.778" layer="97">PC14</text>
+<text x="-198.12" y="-38.1" size="1.778" layer="97">PC15</text>
+<text x="-198.12" y="-35.56" size="1.778" layer="97">PC16</text>
+<text x="-198.12" y="-33.02" size="1.778" layer="97">PC17</text>
+<text x="-198.12" y="-30.48" size="1.778" layer="97">PC18</text>
 </plain>
 <instances>
-<instance part="U1" gate="G$1" x="-220.98" y="0"/>
 <instance part="U2" gate="-A" x="-99.06" y="55.88"/>
 <instance part="U2" gate="-B" x="-99.06" y="0"/>
@@
 <instance part="GND31" gate="1" x="-106.68" y="-160.02"/>
 <instance part="JP4" gate="G$1" x="-170.18" y="60.96" rot="R270"/>
+<instance part="U1" gate="G$1" x="-220.98" y="0"/>
 </instances>
 <busses>
@@
 <net name="+3V3" class="0">
 <segment>
-<pinref part="U1" gate="G$1" pin="3.3V"/>
 <pinref part="+3V2" gate="G$1" pin="+3V3"/>
 <wire x1="-241.3" y1="40.64" x2="-251.46" y2="40.64" width="0.1524" layer="91"/>
 <wire x1="-251.46" y1="40.64" x2="-251.46" y2="43.18" width="0.1524" layer="91"/>
+<pinref part="U1" gate="G$1" pin="3.3V"/>
 </segment>
 <segment>
@@
 <pinref part="GND2" gate="1" pin="GND"/>
 <wire x1="-248.92" y1="-53.34" x2="-248.92" y2="-50.8" width="0.1524" layer="91"/>
-<pinref part="U1" gate="G$1" pin="GND@0"/>
 <wire x1="-248.92" y1="-50.8" x2="-248.92" y2="-48.26" width="0.1524" layer="91"/>
 <wire x1="-248.92" y1="-48.26" x2="-248.92" y2="-45.72" width="0.1524" layer="91"/>
@@
 <wire x1="-248.92" y1="-43.18" x2="-248.92" y2="-40.64" width="0.1524" layer="91"/>
 <wire x1="-248.92" y1="-40.64" x2="-241.3" y2="-40.64" width="0.1524" layer="91"/>
-<pinref part="U1" gate="G$1" pin="GND@1"/>
 <wire x1="-241.3" y1="-43.18" x2="-248.92" y2="-43.18" width="0.1524" layer="91"/>
 <junction x="-248.92" y="-43.18"/>
-<pinref part="U1" gate="G$1" pin="GND@2"/>
 <wire x1="-241.3" y1="-45.72" x2="-248.92" y2="-45.72" width="0.1524" layer="91"/>
 <junction x="-248.92" y="-45.72"/>
-<pinref part="U1" gate="G$1" pin="GND@3"/>
 <wire x1="-241.3" y1="-48.26" x2="-248.92" y2="-48.26" width="0.1524" layer="91"/>
 <junction x="-248.92" y="-48.26"/>
-<pinref part="U1" gate="G$1" pin="GND@4"/>
 <wire x1="-241.3" y1="-50.8" x2="-248.92" y2="-50.8" width="0.1524" layer="91"/>
 <junction x="-248.92" y="-50.8"/>
+<pinref part="U1" gate="G$1" pin="GND@4"/>
+<pinref part="U1" gate="G$1" pin="GND@0"/>
+<pinref part="U1" gate="G$1" pin="GND@1"/>
+<pinref part="U1" gate="G$1" pin="GND@2"/>
+<pinref part="U1" gate="G$1" pin="GND@3"/>
 </segment>
 <segment>
@@
 <pinref part="S1" gate="S" pin="3"/>
 <wire x1="-256.54" y1="33.02" x2="-256.54" y2="35.56" width="0.1524" layer="91"/>
-<pinref part="U1" gate="G$1" pin="RESET"/>
 <wire x1="-256.54" y1="35.56" x2="-241.3" y2="35.56" width="0.1524" layer="91"/>
 <junction x="-256.54" y="35.56"/>
+<pinref part="U1" gate="G$1" pin="RESET"/>
 </segment>
 </net>
@@
 <label x="-233.68" y="-149.86" size="1.778" layer="95"/>
 </segment>
+<segment>
+<wire x1="-200.66" y1="0" x2="-187.96" y2="0" width="0.1524" layer="91"/>
+<label x="-187.96" y="0" size="1.778" layer="95"/>
+<pinref part="U1" gate="G$1" pin="33"/>
+</segment>
 </net>
 <net name="N$13" class="0">
@@
 <label x="-233.68" y="-154.94" size="1.778" layer="95"/>
 </segment>
+<segment>
+<wire x1="-200.66" y1="-2.54" x2="-187.96" y2="-2.54" width="0.1524" layer="91"/>
+<label x="-187.96" y="-2.54" size="1.778" layer="95"/>
+<pinref part="U1" gate="G$1" pin="34"/>
+</segment>
 </net>
 <net name="DAC_WS" class="0">
@@
 <label x="-233.68" y="-160.02" size="1.778" layer="95"/>
 </segment>
+<segment>
+<wire x1="-200.66" y1="-5.08" x2="-187.96" y2="-5.08" width="0.1524" layer="91"/>
+<label x="-187.96" y="-5.08" size="1.778" layer="95"/>
+<pinref part="U1" gate="G$1" pin="35"/>
+</segment>
 </net>
 <net name="DAC_DATAI" class="0">
@@
 <label x="-233.68" y="-165.1" size="1.778" layer="95"/>
 </segment>
+<segment>
+<wire x1="-200.66" y1="-7.62" x2="-187.96" y2="-7.62" width="0.1524" layer="91"/>
+<label x="-187.96" y="-7.62" size="1.778" layer="95"/>
+<pinref part="U1" gate="G$1" pin="36"/>
+</segment>
 </net>
 <net name="DAC_SFOR1" class="0">
@@
 <label x="-233.68" y="-170.18" size="1.778" layer="95"/>
 </segment>
+<segment>
+<wire x1="-200.66" y1="-10.16" x2="-187.96" y2="-10.16" width="0.1524" layer="91"/>
+<label x="-187.96" y="-10.16" size="1.778" layer="95"/>
+<pinref part="U1" gate="G$1" pin="37"/>
+</segment>
 </net>
 <net name="DAC_SFOR0" class="0">
@@
 <label x="-233.68" y="-175.26" size="1.778" layer="95"/>
 </segment>
+<segment>
+<wire x1="-200.66" y1="-12.7" x2="-187.96" y2="-12.7" width="0.1524" layer="91"/>
+<label x="-187.96" y="-12.7" size="1.778" layer="95"/>
+<pinref part="U1" gate="G$1" pin="38"/>
+</segment>
 </net>
 <net name="DAC_MUTE" class="0">
@@
 <label x="-233.68" y="-180.34" size="1.778" layer="95"/>
 </segment>
+<segment>
+<wire x1="-200.66" y1="-15.24" x2="-187.96" y2="-15.24" width="0.1524" layer="91"/>
+<label x="-187.96" y="-15.24" size="1.778" layer="95"/>
+<pinref part="U1" gate="G$1" pin="39"/>
+</segment>
 </net>
 <net name="DAC_DEEM" class="0">
@@
 <label x="-233.68" y="-185.42" size="1.778" layer="95"/>
 </segment>
+<segment>
+<wire x1="-200.66" y1="-17.78" x2="-187.96" y2="-17.78" width="0.1524" layer="91"/>
+<label x="-187.96" y="-17.78" size="1.778" layer="95"/>
+<pinref part="U1" gate="G$1" pin="40"/>
+</segment>
 </net>
 <net name="DAC_PCS" class="0">
@@
 <wire x1="-200.66" y1="-190.5" x2="-215.9" y2="-190.5" width="0.1524" layer="91"/>
 <label x="-233.68" y="-190.5" size="1.778" layer="95"/>
+</segment>
+<segment>
+<wire x1="-200.66" y1="-20.32" x2="-187.96" y2="-20.32" width="0.1524" layer="91"/>
+<label x="-187.96" y="-20.32" size="1.778" layer="95"/>
+<pinref part="U1" gate="G$1" pin="41"/>
 </segment>
 </net>
@@
 <label x="-15.24" y="-172.72" size="1.778" layer="95"/>
 </segment>
+<segment>
+<wire x1="-200.66" y1="-45.72" x2="-187.96" y2="-45.72" width="0.1524" layer="91"/>
+<label x="-187.96" y="-45.72" size="1.778" layer="95"/>
+<pinref part="U1" gate="G$1" pin="51"/>
+</segment>
 </net>
 <net name="ADC_PWON" class="0">
@@
 <label x="-15.24" y="-177.8" size="1.778" layer="95"/>
 </segment>
+<segment>
+<wire x1="-200.66" y1="-43.18" x2="-187.96" y2="-43.18" width="0.1524" layer="91"/>
+<label x="-187.96" y="-43.18" size="1.778" layer="95"/>
+<pinref part="U1" gate="G$1" pin="50"/>
+</segment>
 </net>
 <net name="ADC_SYSCLK" class="0">
@@
 <wire x1="2.54" y1="-182.88" x2="0" y2="-182.88" width="0.1524" layer="91"/>
 <label x="-15.24" y="-182.88" size="1.778" layer="95"/>
+</segment>
+<segment>
+<wire x1="-200.66" y1="-40.64" x2="-187.96" y2="-40.64" width="0.1524" layer="91"/>
+<label x="-187.96" y="-40.64" size="1.778" layer="95"/>
+<pinref part="U1" gate="G$1" pin="49"/>
 </segment>
 </net>
@@
 <label x="38.1" y="-157.48" size="1.778" layer="95"/>
 </segment>
+<segment>
+<wire x1="-200.66" y1="-38.1" x2="-187.96" y2="-38.1" width="0.1524" layer="91"/>
+<label x="-187.96" y="-38.1" size="1.778" layer="95"/>
+<pinref part="U1" gate="G$1" pin="48"/>
+</segment>
 </net>
 <net name="ADC_DATAO" class="0">
@@
 <label x="38.1" y="-162.56" size="1.778" layer="95"/>
 </segment>
+<segment>
+<wire x1="-200.66" y1="-35.56" x2="-187.96" y2="-35.56" width="0.1524" layer="91"/>
+<label x="-187.96" y="-35.56" size="1.778" layer="95"/>
+<pinref part="U1" gate="G$1" pin="47"/>
+</segment>
 </net>
 <net name="ADC_WS" class="0">
@@
 <label x="38.1" y="-167.64" size="1.778" layer="95"/>
 </segment>
+<segment>
+<wire x1="-200.66" y1="-33.02" x2="-187.96" y2="-33.02" width="0.1524" layer="91"/>
+<label x="-187.96" y="-33.02" size="1.778" layer="95"/>
+<pinref part="U1" gate="G$1" pin="46"/>
+</segment>
 </net>
 <net name="ADC_BCK" class="0">
@@
 <wire x1="35.56" y1="-172.72" x2="38.1" y2="-172.72" width="0.1524" layer="91"/>
 <label x="38.1" y="-172.72" size="1.778" layer="95"/>
+</segment>
+<segment>
+<wire x1="-200.66" y1="-30.48" x2="-187.96" y2="-30.48" width="0.1524" layer="91"/>
+<label x="-187.96" y="-30.48" size="1.778" layer="95"/>
+<pinref part="U1" gate="G$1" pin="45"/>
 </segment>
 </net>
@@
 </sheet>
 </sheets>
+<errors>
+</errors>
 </schematic>
 </drawing>
